File: hardware/eagle/liftsensor.brd (EAGLE design)
At the start: 25.4 x 53.3 mm, 7 parts, among them U1 ADXL335

Commit message: Update Eagle designs
Parts:
- added TP1, TP2, TP3, TP4, TP5, TP6, TP7: TEST-POINT3, SparkFun-Connectors:PAD.03X.03
- moved C4 2.54 mm to (17.1, 26.7)
- moved C1 1.27 mm to (7.62, 19.7), turned to 90 degrees
- moved C3 1.27 mm to (7.62, 27.3)
- moved U1 1.27 mm to (12.7, 27.3)
Connections:
- net N$1 renamed VBAT
- removed net N$2: C2.2, EL.11, U1.10
- removed net N$3: C3.2, EL.10, U1.8
- removed net N$5: C1.2, EL.12, U1.12
- new net A0: C1.2, EL.12, TP3.P$1, U1.12
- new net A1: C2.2, EL.11, TP4.P$1, U1.10
- new net A2: C3.2, EL.10, TP5.P$1, U1.8
- new net RX: EL.4, TP6.P$1
- new net TX: EL.3, TP7.P$1
- net GND: now also TP1.P$1
- net VCC_2: now also TP2.P$1
Routing:
- net A0: track 0.00 -> 16.2 mm, vias 0 -> 1
- net A1: track 0.00 -> 13.2 mm, vias 0 -> 1
- net VCC_2: track 28.8 -> 41.9 mm, vias 0 -> 1
- net N$5: track 12.4 -> 0.00 mm
- net A2: track 0.00 -> 11.4 mm, vias 0 -> 1
- net N$2: track 9.11 -> 0.00 mm
- net N$3: track 6.38 -> 0.00 mm
- net TX: track 0.00 -> 5.08 mm, vias 0 -> 1
- net RX: track 0.00 -> 5.08 mm, vias 0 -> 1
- added copper zone on layer 16, net GND
Other:
- board text added: "3.3V"
- board text added: "A0"
- board text added: "A1"
- board text added: "A2"
- board text added: "GND"
- board text added: "RX"
- board text added: "TX"
- board text added: "accessibility.cloud elevator sensor v0.0.3"
- board text removed: "accessibility.cloud elevator sensor v0.0.2"

Commit message: Update hardware design with fixes, add ordered gerber files
Parts:
- C1, C2, C3, C4: device SparkFun-Capacitors:0402 -> SparkFun-Capacitors:0603
- moved C1 3.59 mm to (10.2, 17.1)
- moved C2 1.80 mm to (8.89, 22.2), turned to 90 degrees
Routing:
- net A0: track 16.2 -> 19.7 mm
- net VCC_2: track 41.9 -> 39.0 mm, vias 1 -> 0
- net TX: vias 1 -> 0
- net RX: vias 1 -> 0
- added copper zone on layer 1, net N$1
Other:
- board size 25.4 x 53.3 mm -> 25.4 x 49.5 mm
- board text added: "Projekt Elevate Sensor v0.0.4"
- board text removed: "accessibility.cloud elevator sensor v0.0.3"
