File: hardware/eagle/liftsensor.sch (EAGLE design)
At the start: 7 parts, among them U1 ADXL335

Commit message: Update Eagle designs
Parts:
- added TP1, TP2, TP3, TP4, TP5, TP6, TP7: TEST-POINT3, SparkFun-Connectors:TEST-POINT3
Connections:
- net N$1 renamed VBAT
- removed net N$2: C2.2, EL.A1, U1.YOUT
- removed net N$3: C3.2, EL.A2, U1.ZOUT
- removed net N$5: C1.2, EL.A0, U1.XOUT
- new net A0: C1.2, EL.A0, TP3.1, U1.XOUT
- new net A1: C2.2, EL.A1, TP4.1, U1.YOUT
- new net A2: C3.2, EL.A2, TP5.1, U1.ZOUT
- new net RX: EL.RX, TP6.1
- new net TX: EL.TX, TP7.1
- net GND: now also TP1.1
- net VCC_2: now also TP2.1
Other:
- moved on the sheet: C1, C2, U1
Changed lines of the file:
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@@
 <part name="C3" library="SparkFun-Capacitors" library_urn="urn:adsk.eagle:library:510" deviceset="0.1UF" device="-0402-16V-10%" package3d_urn="urn:adsk.eagle:package:37413/1" value="0.1uF"/>
 <part name="C4" library="SparkFun-Capacitors" library_urn="urn:adsk.eagle:library:510" deviceset="0.1UF" device="-0402-16V-10%" package3d_urn="urn:adsk.eagle:package:37413/1" value="0.1uF"/>
+<part name="GND8" library="SparkFun-PowerSymbols" library_urn="urn:adsk.eagle:library:530" deviceset="GND" device=""/>
+<part name="SUPPLY4" library="SparkFun-PowerSymbols" library_urn="urn:adsk.eagle:library:530" deviceset="VCC_2" device=""/>
+<part name="TP1" library="SparkFun-Connectors" library_urn="urn:adsk.eagle:library:513" deviceset="TEST-POINT" device="3" package3d_urn="urn:adsk.eagle:package:38286/1"/>
+<part name="TP2" library="SparkFun-Connectors" library_urn="urn:adsk.eagle:library:513" deviceset="TEST-POINT" device="3" package3d_urn="urn:adsk.eagle:package:38286/1"/>
+<part name="TP3" library="SparkFun-Connectors" library_urn="urn:adsk.eagle:library:513" deviceset="TEST-POINT" device="3" package3d_urn="urn:adsk.eagle:package:38286/1"/>
+<part name="TP4" library="SparkFun-Connectors" library_urn="urn:adsk.eagle:library:513" deviceset="TEST-POINT" device="3" package3d_urn="urn:adsk.eagle:package:38286/1"/>
+<part name="TP5" library="SparkFun-Connectors" library_urn="urn:adsk.eagle:library:513" deviceset="TEST-POINT" device="3" package3d_urn="urn:adsk.eagle:package:38286/1"/>
+<part name="TP6" library="SparkFun-Connectors" library_urn="urn:adsk.eagle:library:513" deviceset="TEST-POINT" device="3" package3d_urn="urn:adsk.eagle:package:38286/1"/>
+<part name="TP7" library="SparkFun-Connectors" library_urn="urn:adsk.eagle:library:513" deviceset="TEST-POINT" device="3" package3d_urn="urn:adsk.eagle:package:38286/1"/>
 </parts>
 <sheets>
@@
 <instances>
 <instance part="EL" gate="G$1" x="35.56" y="40.64"/>
-<instance part="U1" gate="G$1" x="-22.86" y="30.48"/>
-<instance part="GND1" gate="1" x="-7.62" y="50.8" rot="R180"/>
-<instance part="GND2" gate="1" x="-2.54" y="50.8" rot="R180"/>
+<instance part="U1" gate="G$1" x="-27.94" y="30.48"/>
+<instance part="GND1" gate="1" x="-12.7" y="50.8" rot="R180"/>
+<instance part="GND2" gate="1" x="-5.08" y="50.8" rot="R180"/>
 <instance part="GND3" gate="1" x="2.54" y="50.8" rot="R180"/>
 <instance part="GND4" gate="1" x="-60.96" y="53.34" rot="R180"/>
 <instance part="GND5" gate="1" x="68.58" y="71.12"/>
-<instance part="GND6" gate="1" x="7.62" y="81.28"/>
-<instance part="GND7" gate="1" x="-35.56" y="10.16"/>
+<instance part="GND6" gate="1" x="5.08" y="76.2"/>
+<instance part="GND7" gate="1" x="-40.64" y="10.16"/>
 <instance part="SUPPLY1" gate="G$1" x="-60.96" y="43.18" rot="R180"/>
-<instance part="SUPPLY2" gate="G$1" x="-35.56" y="50.8"/>
+<instance part="SUPPLY2" gate="G$1" x="-40.64" y="50.8"/>
 <instance part="SUPPLY3" gate="G$1" x="68.58" y="83.82"/>
 <instance part="JP1" gate="G$1" x="88.9" y="78.74" rot="R180"/>
-<instance part="C1" gate="G$1" x="-7.62" y="43.18"/>
-<instance part="C2" gate="G$1" x="-2.54" y="43.18"/>
+<instance part="C1" gate="G$1" x="-12.7" y="43.18"/>
+<instance part="C2" gate="G$1" x="-5.08" y="43.18"/>
 <instance part="C3" gate="G$1" x="2.54" y="43.18"/>
 <instance part="C4" gate="G$1" x="-60.96" y="45.72"/>
+<instance part="GND8" gate="1" x="81.28" y="55.88" rot="R180"/>
+<instance part="SUPPLY4" gate="G$1" x="81.28" y="43.18"/>
+<instance part="TP1" gate="G$1" x="88.9" y="53.34"/>
+<instance part="TP2" gate="G$1" x="88.9" y="43.18"/>
+<instance part="TP3" gate="G$1" x="88.9" y="27.94"/>
+<instance part="TP4" gate="G$1" x="88.9" y="17.78"/>
+<instance part="TP5" gate="G$1" x="88.9" y="7.62"/>
+<instance part="TP6" gate="G$1" x="88.9" y="-7.62"/>
+<instance part="TP7" gate="G$1" x="88.9" y="-17.78"/>
 </instances>
 <busses>
@@
 <pinref part="GND6" gate="1" pin="GND"/>
 <pinref part="EL" gate="G$1" pin="GND@2"/>
-<wire x1="7.62" y1="83.82" x2="17.78" y2="78.74" width="0.1524" layer="91"/>
+<wire x1="5.08" y1="78.74" x2="17.78" y2="78.74" width="0.1524" layer="91"/>
 </segment>
 <segment>
@@
 <pinref part="GND7" gate="1" pin="GND"/>
 <pinref part="U1" gate="G$1" pin="COM@7"/>
-<wire x1="-35.56" y1="12.7" x2="-35.56" y2="22.86" width="0.1524" layer="91"/>
+<wire x1="-40.64" y1="12.7" x2="-40.64" y2="22.86" width="0.1524" layer="91"/>
 <pinref part="U1" gate="G$1" pin="COM@6"/>
-<wire x1="-35.56" y1="22.86" x2="-35.56" y2="25.4" width="0.1524" layer="91"/>
-<junction x="-35.56" y="22.86"/>
+<wire x1="-40.64" y1="22.86" x2="-40.64" y2="25.4" width="0.1524" layer="91"/>
+<junction x="-40.64" y="22.86"/>
 <pinref part="U1" gate="G$1" pin="COM@5"/>
-<wire x1="-35.56" y1="25.4" x2="-35.56" y2="27.94" width="0.1524" layer="91"/>
-<junction x="-35.56" y="25.4"/>
+<wire x1="-40.64" y1="25.4" x2="-40.64" y2="27.94" width="0.1524" layer="91"/>
+<junction x="-40.64" y="25.4"/>
 <pinref part="U1" gate="G$1" pin="COM@3"/>
-<wire x1="-35.56" y1="27.94" x2="-35.56" y2="30.48" width="0.1524" layer="91"/>
-<junction x="-35.56" y="27.94"/>
+<wire x1="-40.64" y1="27.94" x2="-40.64" y2="30.48" width="0.1524" layer="91"/>
+<junction x="-40.64" y="27.94"/>
+</segment>
+<segment>
+<pinref part="GND8" gate="1" pin="GND"/>
+<pinref part="TP1" gate="G$1" pin="1"/>
+<wire x1="81.28" y1="53.34" x2="88.9" y2="53.34" width="0.1524" layer="91"/>
 </segment>
 </net>
@@
 <pinref part="U1" gate="G$1" pin="VS@14"/>
 <pinref part="U1" gate="G$1" pin="VS@15"/>
-<wire x1="-35.56" y1="35.56" x2="-35.56" y2="38.1" width="0.1524" layer="91"/>
+<wire x1="-40.64" y1="35.56" x2="-40.64" y2="38.1" width="0.1524" layer="91"/>
 <pinref part="SUPPLY2" gate="G$1" pin="VCC_2"/>
-<wire x1="-35.56" y1="38.1" x2="-35.56" y2="50.8" width="0.1524" layer="91"/>
-<junction x="-35.56" y="38.1"/>
+<wire x1="-40.64" y1="38.1" x2="-40.64" y2="50.8" width="0.1524" layer="91"/>
+<junction x="-40.64" y="38.1"/>
 </segment>
 <segment>
@@
 <wire x1="53.34" y1="83.82" x2="68.58" y2="83.82" width="0.1524" layer="91"/>
 </segment>
-</net>
-<net name="N$2" class="0">
+<segment>
+<pinref part="SUPPLY4" gate="G$1" pin="VCC_2"/>
+<wire x1="88.9" y1="43.18" x2="81.28" y2="43.18" width="0.1524" layer="91"/>
+<pinref part="TP2" gate="G$1" pin="1"/>
+</segment>
+</net>
+<net name="A1" class="0">
 <segment>
 <pinref part="U1" gate="G$1" pin="YOUT"/>
 <pinref part="EL" gate="G$1" pin="A1"/>
 <wire x1="17.78" y1="33.02" x2="15.24" y2="35.56" width="0.1524" layer="91"/>
-<wire x1="15.24" y1="35.56" x2="-2.54" y2="35.56" width="0.1524" layer="91"/>
+<wire x1="15.24" y1="35.56" x2="-5.08" y2="35.56" width="0.1524" layer="91"/>
 <pinref part="C2" gate="G$1" pin="2"/>
-<wire x1="-2.54" y1="35.56" x2="-10.16" y2="35.56" width="0.1524" layer="91"/>
-<wire x1="-2.54" y1="40.64" x2="-2.54" y2="35.56" width="0.1524" layer="91"/>
-<junction x="-2.54" y="35.56"/>
-</segment>
-</net>
-<net name="N$3" class="0">
+<wire x1="-5.08" y1="35.56" x2="-15.24" y2="35.56" width="0.1524" layer="91"/>
+<wire x1="-5.08" y1="40.64" x2="-5.08" y2="35.56" width="0.1524" layer="91"/>
+<junction x="-5.08" y="35.56"/>
+</segment>
+<segment>
+<wire x1="88.9" y1="17.78" x2="81.28" y2="17.78" width="0.1524" layer="91"/>
+<label x="78.74" y="20.32" size="1.778" layer="95"/>
+<pinref part="TP4" gate="G$1" pin="1"/>
+</segment>
+</net>
+<net name="A2" class="0">
 <segment>
 <pinref part="U1" gate="G$1" pin="ZOUT"/>
 <wire x1="5.08" y1="33.02" x2="2.54" y2="33.02" width="0.1524" layer="91"/>
-<wire x1="2.54" y1="33.02" x2="-10.16" y2="33.02" width="0.1524" layer="91"/>
+<wire x1="2.54" y1="33.02" x2="-15.24" y2="33.02" width="0.1524" layer="91"/>
 <wire x1="5.08" y1="33.02" x2="10.16" y2="38.1" width="0.1524" layer="91"/>
 <pinref part="EL" gate="G$1" pin="A2"/>
@@
 <junction x="2.54" y="33.02"/>
 </segment>
-</net>
-<net name="N$5" class="0">
+<segment>
+<wire x1="88.9" y1="7.62" x2="81.28" y2="7.62" width="0.1524" layer="91"/>
+<label x="78.74" y="10.16" size="1.778" layer="95"/>
+<pinref part="TP5" gate="G$1" pin="1"/>
+</segment>
+</net>
+<net name="A0" class="0">
 <segment>
 <pinref part="U1" gate="G$1" pin="XOUT"/>
-<wire x1="-10.16" y1="38.1" x2="-7.62" y2="38.1" width="0.1524" layer="91"/>
-<wire x1="-7.62" y1="38.1" x2="5.08" y2="38.1" width="0.1524" layer="91"/>
+<wire x1="-15.24" y1="38.1" x2="-12.7" y2="38.1" width="0.1524" layer="91"/>
+<wire x1="-12.7" y1="38.1" x2="5.08" y2="38.1" width="0.1524" layer="91"/>
 <wire x1="5.08" y1="38.1" x2="15.24" y2="27.94" width="0.1524" layer="91"/>
 <pinref part="EL" gate="G$1" pin="A0"/>
 <wire x1="15.24" y1="27.94" x2="17.78" y2="27.94" width="0.1524" layer="91"/>
 <pinref part="C1" gate="G$1" pin="2"/>
-<wire x1="-7.62" y1="40.64" x2="-7.62" y2="38.1" width="0.1524" layer="91"/>
-<junction x="-7.62" y="38.1"/>
-</segment>
-</net>
-<net name="N$1" class="0">
+<wire x1="-12.7" y1="40.64" x2="-12.7" y2="38.1" width="0.1524" layer="91"/>
+<junction x="-12.7" y="38.1"/>
+</segment>
+<segment>
+<wire x1="88.9" y1="27.94" x2="81.28" y2="27.94" width="0.1524" layer="91"/>
+<label x="78.74" y="30.48" size="1.778" layer="95"/>
+<pinref part="TP3" gate="G$1" pin="1"/>
+</segment>
+</net>
+<net name="VBAT" class="0">
 <segment>
 <pinref part="EL" gate="G$1" pin="VBAT"/>
@@
 </segment>
 </net>
+<net name="RX" class="0">
+<segment>
+<pinref part="EL" gate="G$1" pin="RX"/>
+<wire x1="17.78" y1="68.58" x2="15.24" y2="68.58" width="0.1524" layer="91"/>
+</segment>
+<segment>
+<wire x1="88.9" y1="-7.62" x2="81.28" y2="-7.62" width="0.1524" layer="91"/>
+<label x="78.74" y="-5.08" size="1.778" layer="95"/>
+<pinref part="TP6" gate="G$1" pin="1"/>
+</segment>
+</net>
+<net name="TX" class="0">
+<segment>
+<pinref part="EL" gate="G$1" pin="TX"/>
+<wire x1="17.78" y1="73.66" x2="15.24" y2="73.66" width="0.1524" layer="91"/>
+</segment>
+<segment>
+<wire x1="88.9" y1="-17.78" x2="81.28" y2="-17.78" width="0.1524" layer="91"/>
+<label x="78.74" y="-15.24" size="1.778" layer="95"/>
+<pinref part="TP7" gate="G$1" pin="1"/>
+</segment>
+</net>

Commit message: Update hardware design with fixes, add ordered gerber files
Parts:
- C1, C2, C3, C4: device SparkFun-Capacitors:0.1UF-0402-16V-10% -> SparkFun-Capacitors:0.1UF-0603-25V-5%
Changed lines of the file:
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@@
 <part name="SUPPLY3" library="SparkFun-PowerSymbols" library_urn="urn:adsk.eagle:library:530" deviceset="VCC_2" device=""/>
 <part name="JP1" library="pinhead" library_urn="urn:adsk.eagle:library:325" deviceset="PINHD-1X2" device="/90" package3d_urn="urn:adsk.eagle:package:22437/2"/>
-<part name="C1" library="SparkFun-Capacitors" library_urn="urn:adsk.eagle:library:510" deviceset="0.1UF" device="-0402-16V-10%" package3d_urn="urn:adsk.eagle:package:37413/1" value="0.1uF"/>
-<part name="C2" library="SparkFun-Capacitors" library_urn="urn:adsk.eagle:library:510" deviceset="0.1UF" device="-0402-16V-10%" package3d_urn="urn:adsk.eagle:package:37413/1" value="0.1uF"/>
-<part name="C3" library="SparkFun-Capacitors" library_urn="urn:adsk.eagle:library:510" deviceset="0.1UF" device="-0402-16V-10%" package3d_urn="urn:adsk.eagle:package:37413/1" value="0.1uF"/>
-<part name="C4" library="SparkFun-Capacitors" library_urn="urn:adsk.eagle:library:510" deviceset="0.1UF" device="-0402-16V-10%" package3d_urn="urn:adsk.eagle:package:37413/1" value="0.1uF"/>
+<part name="C1" library="SparkFun-Capacitors" library_urn="urn:adsk.eagle:library:510" deviceset="0.1UF" device="-0603-25V-5%" package3d_urn="urn:adsk.eagle:package:37414/1" value="0.1uF"/>
+<part name="C2" library="SparkFun-Capacitors" library_urn="urn:adsk.eagle:library:510" deviceset="0.1UF" device="-0603-25V-5%" package3d_urn="urn:adsk.eagle:package:37414/1" value="0.1uF"/>
+<part name="C3" library="SparkFun-Capacitors" library_urn="urn:adsk.eagle:library:510" deviceset="0.1UF" device="-0603-25V-5%" package3d_urn="urn:adsk.eagle:package:37414/1" value="0.1uF"/>
+<part name="C4" library="SparkFun-Capacitors" library_urn="urn:adsk.eagle:library:510" deviceset="0.1UF" device="-0603-25V-5%" package3d_urn="urn:adsk.eagle:package:37414/1" value="0.1uF"/>
 <part name="GND8" library="SparkFun-PowerSymbols" library_urn="urn:adsk.eagle:library:530" deviceset="GND" device=""/>
 <part name="SUPPLY4" library="SparkFun-PowerSymbols" library_urn="urn:adsk.eagle:library:530" deviceset="VCC_2" device=""/>
